Commit message: first commit

File: description/robot.urdf.xacro (robot description, xacro)
@@ -1,11 +1,12 @@
 <?xml version="1.0"?>
 <robot xmlns:xacro="http://www.ros.org/wiki/xacro"  name="robot">
+    <xacro:arg name="use_ros2_control" default="true"/>
     <xacro:include filename="robot_core.xacro" />
-<<<<<<< HEAD
-    <!-- <xacro:include filename="gazebo_control.xacro" /> -->
-    <xacro:include filename="ros2_control.xacro" />
-=======
-    <xacro:include filename="gazebo_control.xacro" />
->>>>>>> e2c564ac18a9e73b7e968ace8e992ae9022791a9
+    <xacro:if value="$(arg use_ros2_control)">
+        <xacro:include filename="ros2_control.xacro" />
+    </xacro:if>
+    <xacro:unless value="$(arg use_ros2_control)">
+        <xacro:include filename="gazebo_control.xacro" />
+    </xacro:unless>
     <xacro:include filename="lidar.xacro" />
 </robot>

File: description/robot_core.xacro (robot description, xacro)
@@ -63,5 +63,5 @@
     <collision>
         <geometry>
-            <cylinder length="0.04" radius="0.05" />/>
+            <sphere radius="0.05" />/>
         </geometry>
         <material name="blue"/>
@@ -90,5 +90,5 @@
     <collision>
         <geometry>
-            <cylinder length="0.04" radius="0.05" />/>
+            <sphere radius="0.05" />/>
         </geometry>
         <material name="blue"/>

File: description/ros2_control.xacro (robot description, xacro)
@@ -1,4 +1,32 @@
 <?xml version="1.0"?>
 <robot xmlns:xacro="http://www.ros.org/wiki/xacro">
+<!--<ros2_control name="RealRobot" type="system">
+    <hardware>
+        <plugin>diffdrive_arduino/DiffDriveArduino</plugin>
+        <param name="left_wheel_name">left_wheel_joint</param>
+        <param name="right_wheel_name">right_wheel_joint</param>
+        <param name="loop_rate">30</param>
+        <param name="device">/dev/ttyUSB0</param>
+        <param name="baud_rate">57600</param>
+        <param name="timeout">1000</param>
+        <param name="enc_counts_per_rev">8100</param>
+    </hardware>
+    <joint name="left_wheel_joint">
+        <command_interface name="velocity">
+            <param name="min">-10</param>
+            <param name="max">10</param>
+        </command_interface>
+        <state_interface name="position" />
+        <state_interface name="velocity" />
+    </joint>
+    <joint name="right_wheel_joint">
+        <command_interface name="velocity">
+            <param name="min">-10</param>
+            <param name="max">10</param>
+        </command_interface>
+        <state_interface name="velocity" />
+        <state_interface name="position" />
+    </joint>
+</ros2_control> -->
 <ros2_control name="GazeboSystem" type="system">
     <hardware>

Commit message: first commit

File: description/robot.urdf.xacro (robot description, xacro)
@@ -2,4 +2,5 @@
 <robot xmlns:xacro="http://www.ros.org/wiki/xacro"  name="robot">
     <xacro:arg name="use_ros2_control" default="true"/>
+    <xacro:arg name="sim_mode" default="false"/>
     <xacro:include filename="robot_core.xacro" />
     <xacro:if value="$(arg use_ros2_control)">

File: description/robot_core.xacro (robot description, xacro)
@@ -33,4 +33,12 @@
     <!-- BASE LINK -->
     <link name="base_link">
+    </link>
+    <!-- BASE_FOOTPRINT LINK -->
+    <joint name="base_footprint_joint" type="fixed">
+        <parent link="base_link"/>
+        <child link="base_footprint"/>
+        <origin xyz="0 0 0" rpy="0 0 0"/>
+    </joint>
+    <link name="base_footprint">
     </link>
     <!-- CHASSIS LINK -->

File: description/ros2_control.xacro (robot description, xacro)
@@ -1,56 +1,61 @@
 <?xml version="1.0"?>
 <robot xmlns:xacro="http://www.ros.org/wiki/xacro">
-<ros2_control name="RealRobot" type="system">
-    <hardware>
-        <plugin>diffdrive_arduino/DiffDriveArduino</plugin>
-        <param name="left_wheel_name">left_wheel_joint</param>
-        <param name="right_wheel_name">right_wheel_joint</param>
-        <param name="loop_rate">30</param>
-        <param name="device">/dev/ttyUSB0</param>
-        <param name="baud_rate">57600</param>
-        <param name="timeout">1000</param>
-        <param name="enc_counts_per_rev">8100</param>
-    </hardware>
-    <joint name="left_wheel_joint">
-        <command_interface name="velocity">
-            <param name="min">-10</param>
-            <param name="max">10</param>
-        </command_interface>
-        <state_interface name="position" />
-        <state_interface name="velocity" />
-    </joint>
-    <joint name="right_wheel_joint">
-        <command_interface name="velocity">
-            <param name="min">-10</param>
-            <param name="max">10</param>
-        </command_interface>
-        <state_interface name="velocity" />
-        <state_interface name="position" />
-    </joint>
-</ros2_control>
- <!-- <ros2_control name="GazeboSystem" type="system">
-    <hardware>
-        <plugin>gazebo_ros2_control/GazeboSystem</plugin>
-    </hardware>
-    <joint name="left_wheel_joint">
-        <command_interface name="velocity">
-            <param name="min">-10</param>
-            <param name="max">10</param>
-        </command_interface>
-        <state_interface name="position" />
-        <state_interface name="velocity" />
-    </joint>
-    <joint name="right_wheel_joint">
-        <command_interface name="velocity">
-            <param name="min">-10</param>
-            <param name="max">10</param>
-        </command_interface>
-        <state_interface name="velocity" />
-        <state_interface name="position" />
-    </joint>
-</ros2_control> -->
+<xacro:unless value="$(arg sim_mode)">
+    <ros2_control name="RealRobot" type="system">
+        <hardware>
+            <plugin>diffdrive_arduino/DiffDriveArduino</plugin>
+            <param name="left_wheel_name">left_wheel_joint</param>
+            <param name="right_wheel_name">right_wheel_joint</param>
+            <param name="loop_rate">30</param>
+            <param name="device">/dev/ttyUSB0</param>
+            <param name="baud_rate">57600</param>
+            <param name="timeout">1000</param>
+            <param name="enc_counts_per_rev">8100</param>
+        </hardware>
+        <joint name="left_wheel_joint">
+            <command_interface name="velocity">
+                <param name="min">-10</param>
+                <param name="max">10</param>
+            </command_interface>
+            <state_interface name="position" />
+            <state_interface name="velocity" />
+        </joint>
+        <joint name="right_wheel_joint">
+            <command_interface name="velocity">
+                <param name="min">-10</param>
+                <param name="max">10</param>
+            </command_interface>
+            <state_interface name="velocity" />
+            <state_interface name="position" />
+        </joint>
+    </ros2_control>
+</xacro:unless>
+<xacro:if value="$(arg sim_mode)">
+        <ros2_control name="GazeboSystem" type="system">
+            <hardware>
+                <plugin>gazebo_ros2_control/GazeboSystem</plugin>
+            </hardware>
+            <joint name="left_wheel_joint">
+                <command_interface name="velocity">
+                    <param name="min">-10</param>
+                    <param name="max">10</param>
+                </command_interface>
+                <state_interface name="velocity"/>
+                <state_interface name="position"/>
+            </joint>
+            <joint name="right_wheel_joint">
+                <command_interface name="velocity">
+                    <param name="min">-10</param>
+                    <param name="max">10</param>
+                </command_interface>
+                <state_interface name="velocity"/>
+                <state_interface name="position"/>
+            </joint>
+        </ros2_control>
+    </xacro:if>
 <gazebo>
     <plugin name="gazebo_ros2_control" filename="libgazebo_ros2_control.so" >
-     <parameters>$(find my_bot)/config/my_controllers.yaml</parameters>
+        <parameters>$(find my_bot)/config/my_controllers.yaml</parameters>
+        <parameters>$(find my_bot)/config/gaz_ros2_ctl_sim.yaml</parameters>
     </plugin>
 </gazebo>

Commit message: first commit

File: description/robot.urdf.xacro (robot description, xacro)
@@ -11,4 +11,4 @@
     </xacro:unless>
     <xacro:include filename="lidar.xacro" />
-    <!-- <xacro:include filename="depth_camera.xacro" /> -->
+    <xacro:include filename="camera.xacro" />
 </robot>

File: description/robot_core.xacro (robot description, xacro)
@@ -9,5 +9,5 @@
     <xacro:property name="wheel_thickness" value="0.026"/>
     <xacro:property name="wheel_mass" value="0.05"/>
-    <xacro:property name="wheel_offset_x" value="0.226"/>
+    <xacro:property name="wheel_offset_x" value="0.285"/>
     <xacro:property name="wheel_offset_y" value="0.1485"/>
     <xacro:property name="wheel_offset_z" value="0.01"/>
